File: eagle/zigbee_dimmer/zigbee-dimmer.sch (EAGLE design)
At the start: 0 parts

Commit message: eagle updated
Parts:
- added J1: (no value), SparkFun-Connectors:JST_2MM_MALE
- added JP1: (no value), zigbee-dimmer-libs:DIMMER_PINSSMD_180
- added U1: POLOLU-ASTAR-MICRO, zigbee-dimmer-libs:POLOLU-ASTAR-MICRO
- added U2: CREE_ZIGBEE, zigbee-dimmer-libs:CREE_ZIGBEE
Connections:
- new net 3V3: JP1.4, U1.3V3, U2.VCC
- new net GATE: JP1.2, U1.6
- new net GND: J1.-, JP1.1, U1.GND, U2.GND
- new net ONOFF: U1.8, U2.ON_OFF
- new net PWM: U1.3, U2.PWM
- new net SYNC: JP1.3, U1.2
- new net VCC: J1.+, U1.VIN
